Commit message: Stair climbing commit

File: amr_description/urdf/amr.urdf.xacro (robot description, xacro)
@@ -20,5 +20,5 @@
       </material>
     </visual>
-    <collision>
+    <!--collision>
       <origin
         xyz="0 0 0"
@@ -28,5 +28,5 @@
           filename="package://amr_description/meshes/base_link.stl" scale="0.001 0.001 0.001" />
       </geometry>
-    </collision>
+    </collision-->
     <inertial>
       <origin
@@ -89,5 +89,5 @@
     </inertial>
   </link>
-  <joint name="front_right_link_revolute" type="continuous">
+  <joint name="front_right_link_revolute" type="revolute">
     <parent link="base_link"/>
     <child link="front_link_right_side"/>
@@ -95,4 +95,6 @@
     <axis xyz="0 1 0"/>
     <limit
+      lower="-1.13446"
+      upper="0.750492"
       effort="10000000"
       velocity="10000000" />
@@ -141,5 +143,5 @@
     </inertial>
   </link>
-  <joint name="front_left_link_revolute" type="continuous">
+  <joint name="front_left_link_revolute" type="revolute">
     <parent link="base_link"/>
     <child link="front_link_left_side"/>
@@ -147,4 +149,6 @@
     <axis xyz="0 1 0"/>
     <limit
+      lower="-1.13446"
+      upper="0.750492"
       effort="10000000"
       velocity="10000000" />
@@ -267,4 +271,12 @@
           filename="package://amr_description/meshes/back_wheel_right_side.stl" scale="0.001 0.001 0.001" />
       </geometry>
+      <surface>
+        <friction>
+          <ode>
+            <mu>10.0</mu> <!-- High friction -->
+            <mu2>10.0</mu2>
+          </ode>
+        </friction>
+      </surface>
     </collision>
     <inertial>
@@ -319,4 +331,12 @@
           filename="package://amr_description/meshes/back_wheel_left_side.stl" scale="0.001 0.001 0.001" />
       </geometry>
+      <surface>
+        <friction>
+          <ode>
+            <mu>10.0</mu> <!-- High friction -->
+            <mu2>10.0</mu2>
+          </ode>
+        </friction>
+      </surface>
     </collision>
     <inertial>
@@ -371,4 +391,12 @@
           filename="package://amr_description/meshes/middle_wheel_left_side.stl" scale="0.001 0.001 0.001" />
       </geometry>
+      <surface>
+        <friction>
+          <ode>
+            <mu>10.0</mu> <!-- High friction -->
+            <mu2>10.0</mu2>
+          </ode>
+        </friction>
+      </surface>
     </collision>
     <inertial>
@@ -423,4 +451,12 @@
           filename="package://amr_description/meshes/middle_wheel_right_side.stl" scale="0.001 0.001 0.001" />
       </geometry>
+      <surface>
+        <friction>
+          <ode>
+            <mu>10.0</mu> <!-- High friction -->
+            <mu2>10.0</mu2>
+          </ode>
+        </friction>
+      </surface>
     </collision>
     <inertial>
@@ -475,4 +511,12 @@
           filename="package://amr_description/meshes/front_wheel_left_side.stl" scale="0.001 0.001 0.001" />
       </geometry>
+      <surface>
+        <friction>
+          <ode>
+            <mu>10.0</mu> <!-- High friction -->
+            <mu2>10.0</mu2>
+          </ode>
+        </friction>
+      </surface>
     </collision>
     <inertial>
@@ -527,4 +571,12 @@
           filename="package://amr_description/meshes/front_wheel_right_side.stl" scale="0.001 0.001 0.001" />
       </geometry>
+      <surface>
+        <friction>
+          <ode>
+            <mu>10.0</mu> <!-- High friction -->
+            <mu2>10.0</mu2>
+          </ode>
+        </friction>
+      </surface>
     </collision>
     <inertial>

File: amr_description/urdf/amr_gazebo.xacro (robot description, xacro)
@@ -2,8 +2,14 @@
 <robot name="amr" xmlns:xacro="http://ros.org/wiki/xacro">
     <gazebo reference="back_wheel_right_side">
-        <mu1>100000000000000.0</mu1>
-        <mu2>100000000000000.0</mu2>
-        <kp>10000000000000.0</kp>
-        <kd>10.0</kd>
+  <material>
+    <friction>
+      <mu1>0.9</mu1>
+      <mu2>0.9</mu2>
+    </friction>
+    <surface>
+      <kp>100000.0</kp>
+      <kd>1.0</kd>
+    </surface>
+  </material>
         <minDepth>0.001</minDepth>
         <maxVel>0.1</maxVel>
@@ -11,8 +17,14 @@
     </gazebo>
     <gazebo reference="back_wheel_left_side">
-        <mu1>100000000000000.0</mu1>
-        <mu2>100000000000000.0</mu2>
-        <kp>10000000000000.0</kp>
-        <kd>10.0</kd>
+  <material>
+    <friction>
+      <mu1>0.9</mu1>
+      <mu2>0.9</mu2>
+    </friction>
+    <surface>
+      <kp>100000.0</kp>
+      <kd>1.0</kd>
+    </surface>
+  </material>
         <minDepth>0.001</minDepth>
         <maxVel>0.1</maxVel>
@@ -20,8 +32,14 @@
     </gazebo>
     <gazebo reference="middle_wheel_right_side">
-        <mu1>100000000000000.0</mu1>
-        <mu2>100000000000000.0</mu2>
-        <kp>10000000000000.0</kp>
-        <kd>10.0</kd>
+  <material>
+    <friction>
+      <mu1>0.9</mu1>
+      <mu2>0.9</mu2>
+    </friction>
+    <surface>
+      <kp>100000.0</kp>
+      <kd>1.0</kd>
+    </surface>
+  </material>
         <minDepth>0.001</minDepth>
         <maxVel>0.1</maxVel>
@@ -29,8 +47,14 @@
     </gazebo>
     <gazebo reference="middle_wheel_left_side">
-        <mu1>100000000000000.0</mu1>
-        <mu2>100000000000000.0</mu2>
-        <kp>10000000000000.0</kp>
-        <kd>10.0</kd>
+  <material>
+    <friction>
+      <mu1>0.9</mu1>
+      <mu2>0.9</mu2>
+    </friction>
+    <surface>
+      <kp>100000.0</kp>
+      <kd>1.0</kd>
+    </surface>
+  </material>
         <minDepth>0.001</minDepth>
         <maxVel>0.1</maxVel>
@@ -38,8 +62,14 @@
     </gazebo>
     <gazebo reference="front_wheel_right_side">
-        <mu1>100000000000000.0</mu1>
-        <mu2>100000000000000.0</mu2>
-        <kp>10000000000000.0</kp>
-        <kd>10.0</kd>
+  <material>
+    <friction>
+      <mu1>0.9</mu1>
+      <mu2>0.9</mu2>
+    </friction>
+    <surface>
+      <kp>100000.0</kp>
+      <kd>1.0</kd>
+    </surface>
+  </material>
         <minDepth>0.001</minDepth>
         <maxVel>0.1</maxVel>
@@ -47,8 +77,14 @@
     </gazebo>
     <gazebo reference="front_wheel_left_side">
-        <mu1>100000000000000.0</mu1>
-        <mu2>100000000000000.0</mu2>
-        <kp>10000000000000.0</kp>
-        <kd>10.0</kd>
+  <material>
+    <friction>
+      <mu1>0.9</mu1>
+      <mu2>0.9</mu2>
+    </friction>
+    <surface>
+      <kp>100000.0</kp>
+      <kd>1.0</kd>
+    </surface>
+  </material>
         <minDepth>0.001</minDepth>
         <maxVel>0.1</maxVel>

Commit message: modelled stairs and all componenets stl file added

File: amr_description/urdf/amr.urdf.xacro (robot description, xacro)
@@ -607,3 +607,215 @@
       friction="0.2" />
   </joint>
+  <link name="imu_link">
+    <visual>
+      <geometry>
+        <box size="0.02 0.02 0.005"/>
+      </geometry>
+      <material name="black">
+				<color rgba="0 0 0 1"/>
+			</material>
+    </visual>
+  </link>
+  <joint name="imu_base_joint" type="fixed">
+      <parent link="base_link"/>
+      <child link="imu_link"/>
+      <origin xyz="0 0 0.005" rpy="0 0 0"/>
+      <axis xyz="0 0 0"/>
+  </joint>
+<link
+    name="connector">
+    <visual>
+      <origin
+        xyz="0 0 0"
+        rpy="0 0 0" />
+      <geometry>
+        <mesh
+          filename="package://amr_description/meshes/connector.stl" scale="0.001 0.001 0.001"/>
+      </geometry>
+      <material
+        name="">
+        <color
+          rgba="0.792156862745098 0.819607843137255 0.933333333333333 1" />
+      </material>
+    </visual>
+    <collision>
+      <origin
+        xyz="0 0 0"
+        rpy="0 0 0" />
+      <geometry>
+        <mesh
+          filename="package://amr_description/meshes/connector.stl" scale="0.001 0.001 0.001" />
+      </geometry>
+    </collision>
+    <inertial>
+      <origin
+        xyz="0 0 0.025"
+        rpy="0 0 0" />
+      <mass
+        value="12.076e-3" />
+      <inertia
+        ixx="2.205e-6"
+        ixy="-4.149e-18"
+        ixz="-3.479e-14"
+        iyy="2.451457e-6"
+        iyz="-0.434e-9"
+        izz="3.35403e-7" />
+    </inertial>
+  </link>
+  <joint name="connector_base_joint" type="fixed">
+      <parent link="base_link"/>
+      <child link="connector"/>
+      <origin xyz="0.0685 0 0.022079" rpy="0 0 0"/>
+      <axis xyz="0 0 0"/>
+  </joint>
+  <link
+    name="prism_bottom_tab">
+    <visual>
+      <origin
+        xyz="0 0 0"
+        rpy="0 0 0" />
+      <geometry>
+        <mesh
+          filename="package://amr_description/meshes/prism_bottom_tab.stl" scale="0.001 0.001 0.001"/>
+      </geometry>
+      <material
+        name="">
+        <color
+          rgba="0.792156862745098 0.819607843137255 0.933333333333333 1" />
+      </material>
+    </visual>
+  </link>
+  <joint name="prism_bottom_tab_base_joint" type="fixed">
+      <parent link="base_link"/>
+      <child link="prism_bottom_tab"/>
+      <origin xyz="-0.045604 0 0.005" rpy="0 0 0"/>
+      <axis xyz="0 0 0"/>
+  </joint>
+  <link
+    name="prismatic_joint_bottom_hc">
+    <visual>
+      <origin
+        xyz="0 0 0"
+        rpy="0 0 0" />
+      <geometry>
+        <mesh
+          filename="package://amr_description/meshes/prismatic_joint_bottom_hc.stl" scale="0.001 0.001 0.001"/>
+      </geometry>
+      <material
+        name="">
+        <color
+          rgba="0.792156862745098 0.819607843137255 0.933333333333333 1" />
+      </material>
+    </visual>
+  </link>
+  <joint name="hc_bt_joint" type="fixed">
+      <parent link="prism_bottom_tab"/>
+      <child link="prismatic_joint_bottom_hc"/>
+      <origin xyz="0 0 0.012809" rpy="0 0 0"/>
+      <!--axis xyz="0 1 0"/>
+    <limit
+      effort="10000000"
+      velocity="10000000" />
+    <dynamics
+      damping="0.1"
+      friction="0.2" /-->
+  </joint>
+  <link
+    name="prismatic_joint_top_sc">
+    <visual>
+      <origin
+        xyz="0 0 0"
+        rpy="0 0.7382 0" />
+      <geometry>
+        <mesh
+          filename="package://amr_description/meshes/prismatic_joint_top_sc.stl" scale="0.001 0.001 0.001"/>
+      </geometry>
+      <material
+        name="">
+        <color
+          rgba="0.792156862745098 0.819607843137255 0.933333333333333 1" />
+      </material>
+    </visual>
+  </link>
+  <joint name="sc_hc_joint" type="fixed">
+      <parent link="prismatic_joint_bottom_hc"/>
+      <child link="prismatic_joint_top_sc"/>
+      <origin xyz="0.011825 0 0.005501" rpy="0 -0.7382 0"/>
+      <!--limit effort="1000.0" lower="0.0" upper="0.05" velocity="0.5"/-->
+  </joint>
+  <link
+    name="prism_top_tab">
+    <visual>
+      <origin
+        xyz="0 0 0"
+        rpy="0 0 0" />
+      <geometry>
+        <mesh
+          filename="package://amr_description/meshes/prism_top_tab.stl" scale="0.001 0.001 0.001"/>
+      </geometry>
+      <material
+        name="">
+        <color
+          rgba="0.792156862745098 0.819607843137255 0.933333333333333 1" />
+      </material>
+    </visual>
+  </link>
+  <joint name="top_tab_sc_joint" type="fixed">
+      <parent link="prismatic_joint_top_sc"/>
+      <child link="prism_top_tab"/>
+      <origin xyz="0.068867 0 -0.004082" rpy="0 0.7382 0"/>
+      <!--axis xyz="0 1 0"/>
+      <limit
+        effort="10000000"
+        velocity="10000000" />
+      <dynamics
+        damping="0.1"
+        friction="0.2" /-->
+  </joint>
+  <link
+    name="delivery_box">
+    <visual>
+      <origin
+        xyz="0 0 0"
+        rpy="0 0 0" />
+      <geometry>
+        <mesh
+          filename="package://amr_description/meshes/delivery_box.stl" scale="0.001 0.001 0.001"/>
+      </geometry>
+      <material
+        name="">
+        <color
+          rgba="0.792156862745098 0.819607843137255 0.933333333333333 1" />
+      </material>
+    </visual>
+    <collision>
+      <origin
+        xyz="0 0 0"
+        rpy="0 0 0" />
+      <geometry>
+        <mesh
+          filename="package://amr_description/meshes/delivery_box.stl" scale="0.001 0.001 0.001" />
+      </geometry>
+    </collision>
+    <!--inertial>
+      <origin
+        xyz="0.03 0 0.03"
+        rpy="0 0 0" />
+      <mass
+        value="1.030" />
+      <inertia
+        ixx="7.791e-4"
+        ixy="-0.013e-9"
+        ixz="-1.04741e-7"
+        iyy="8.515e-4"
+        iyz="2.7531e-8"
+        izz="7.801e-4" />
+    </inertial-->
+  </link>
+  <joint name="del_box_connector" type="continuous">
+      <parent link="connector"/>
+      <child link="delivery_box"/>
+      <origin xyz="0 0 0.1" rpy="0 0 0"/>
+      <axis xyz="0 1 0"/>
+  </joint>
 </robot>

File: amr_description/urdf/amr_gazebo.xacro (robot description, xacro)
@@ -96,4 +96,6 @@
                 <parameters>$(find amr_controller)/config/amr_controllers.yaml</parameters>
             </plugin>
+            <plugin filename="ignition-gazebo-imu-system" name="ignition::gazebo::systems::Imu">
+            </plugin>
         <!--/xacro:if-->
         <!--xacro:unless value="$(arg is_ignition)">
@@ -103,3 +105,53 @@
         </xacro:unless-->
     </gazebo>
+    <gazebo reference="imu_link">
+      <sensor name="imu" type="imu">
+       <always_on>true</always_on>
+       <update_rate>50</update_rate>
+       <gz_frame_id> imu_link</gz_frame_id>
+       <topic>imu</topic>
+       <imu>
+        <angular_velocity>
+          <x>
+            <noise type="gaussian">
+              <mean>0.0</mean>
+              <stddev>2e-4</stddev>
+            </noise>
+          </x>
+          <y>
+            <noise type="gaussian">
+              <mean>0.0</mean>
+              <stddev>2e-4</stddev>
+            </noise>
+          </y>
+          <z>
+            <noise type="gaussian">
+              <mean>0.0</mean>
+              <stddev>2e-4</stddev>
+            </noise>
+          </z>
+        </angular_velocity>
+        <linear_acceleration>
+          <x>
+            <noise type="gaussian">
+              <mean>0.0</mean>
+              <stddev>1.7e-2</stddev>
+            </noise>
+          </x>
+          <y>
+            <noise type="gaussian">
+              <mean>0.0</mean>
+              <stddev>1.7e-2</stddev>
+            </noise>
+          </y>
+          <z>
+            <noise type="gaussian">
+              <mean>0.0</mean>
+              <stddev>1.7e-2</stddev>
+            </noise>
+          </z>
+        </linear_acceleration>
+       </imu>
+      </sensor>
+    </gazebo>
 </robot>

Commit message: modelled stairs and all componenets stl file added

File: amr_description/urdf/amr.urdf.xacro (robot description, xacro)
@@ -648,18 +648,4 @@
       </geometry>
     </collision>
-    <inertial>
-      <origin
-        xyz="0 0 0.025"
-        rpy="0 0 0" />
-      <mass
-        value="12.076e-3" />
-      <inertia
-        ixx="2.205e-6"
-        ixy="-4.149e-18"
-        ixz="-3.479e-14"
-        iyy="2.451457e-6"
-        iyz="-0.434e-9"
-        izz="3.35403e-7" />
-    </inertial>
   </link>
   <joint name="connector_base_joint" type="fixed">
@@ -781,27 +767,27 @@
       <geometry>
         <mesh
-          filename="package://amr_description/meshes/delivery_box.stl" scale="0.001 0.001 0.001"/>
-      </geometry>
-      <material
-        name="">
-        <color
-          rgba="0.792156862745098 0.819607843137255 0.933333333333333 1" />
-      </material>
-    </visual>
-    <collision>
-      <origin
-        xyz="0 0 0"
-        rpy="0 0 0" />
-      <geometry>
-        <mesh
-          filename="package://amr_description/meshes/delivery_box.stl" scale="0.001 0.001 0.001" />
-      </geometry>
-    </collision>
-    <!--inertial>
-      <origin
-        xyz="0.03 0 0.03"
-        rpy="0 0 0" />
-      <mass
-        value="1.030" />
+          filename="package://amr_description/meshes/delivery_box_wol.stl" scale="0.001 0.001 0.001"/>
+      </geometry>
+      <material
+        name="">
+        <color
+          rgba="0.792156862745098 0.819607843137255 0.933333333333333 1" />
+      </material>
+    </visual>
+    <collision>
+      <origin
+        xyz="0 0 0"
+        rpy="0 0 0" />
+      <geometry>
+        <mesh
+          filename="package://amr_description/meshes/delivery_box_wol.stl" scale="0.001 0.001 0.001" />
+      </geometry>
+    </collision>
+    <inertial>
+      <origin
+        xyz="0.045 0 0.03"
+        rpy="0 0 0" />
+      <mass
+        value="0.000000001" />
       <inertia
         ixx="7.791e-4"
@@ -811,11 +797,19 @@
         iyz="2.7531e-8"
         izz="7.801e-4" />
-    </inertial-->
-  </link>
-  <joint name="del_box_connector" type="continuous">
+    </inertial>
+  </link>
+  <joint name="del_box_connector" type="revolute">
       <parent link="connector"/>
       <child link="delivery_box"/>
-      <origin xyz="0 0 0.1" rpy="0 0 0"/>
+      <origin xyz="0 0 0.039994" rpy="0 0 0"/>
       <axis xyz="0 1 0"/>
+      <limit
+        lower="0.0"
+        upper="0.890118"
+        effort="10000000"
+        velocity="10000000" />
+      <dynamics
+        damping="0.1"
+        friction="0.2" />
   </joint>
 </robot>
