Commit message: delivery box stabilization added

File: amr_description/urdf/amr.urdf.xacro (robot description, xacro)
@@ -34,5 +34,5 @@
         rpy="0 0 0" />
       <mass
-        value="1.501384" />
+        value="1.001384" />
       <inertia
         ixx="8.726e-3"
@@ -285,5 +285,5 @@
         rpy="0 0 0" />
       <mass
-        value="0.595006" />
+        value="0.295006" />
       <inertia
         ixx="3.284e-4"
@@ -301,5 +301,5 @@
     <axis xyz="0 1 0"/>
     <limit
-      effort="10000000"
+      effort="10000000000"
       velocity="10000000" />
     <dynamics
@@ -345,5 +345,5 @@
         rpy="0 0 0" />
       <mass
-        value="0.595006" />
+        value="0.295006" />
       <inertia
         ixx="3.284e-4"
@@ -361,5 +361,5 @@
     <axis xyz="0 1 0"/>
     <limit
-      effort="10000000"
+      effort="10000000000"
       velocity="10000000" />
     <dynamics
@@ -405,5 +405,5 @@
         rpy="0 0 0" />
       <mass
-        value="0.595006" />
+        value="0.295006" />
       <inertia
         ixx="3.284e-4"
@@ -421,5 +421,5 @@
     <axis xyz="0 1 0"/>
     <limit
-      effort="10000000"
+      effort="10000000000"
       velocity="10000000" />
     <dynamics
@@ -465,5 +465,5 @@
         rpy="0 0 0" />
       <mass
-        value="0.595006" />
+        value="0.295006" />
       <inertia
         ixx="3.284e-4"
@@ -481,5 +481,5 @@
     <axis xyz="0 1 0"/>
     <limit
-      effort="10000000"
+      effort="10000000000"
       velocity="10000000" />
     <dynamics
@@ -525,5 +525,5 @@
         rpy="0 0 0" />
       <mass
-        value="1.030" />
+        value="0.530" />
       <inertia
         ixx="7.791e-4"
@@ -541,5 +541,5 @@
     <axis xyz="0 1 0"/>
     <limit
-      effort="10000000"
+      effort="10000000000"
       velocity="10000000" />
     <dynamics
@@ -585,5 +585,5 @@
         rpy="0 0 0" />
       <mass
-        value="1.030" />
+        value="0.530" />
       <inertia
         ixx="7.791e-4"
@@ -601,5 +601,5 @@
     <axis xyz="0 1 0"/>
     <limit
-      effort="10000000"
+      effort="10000000000"
       velocity="10000000" />
     <dynamics
@@ -805,10 +805,10 @@
       <axis xyz="0 1 0"/>
       <limit
-        lower="0.0"
+        lower="-0.0873"
         upper="0.890118"
         effort="10000000"
         velocity="10000000" />
       <dynamics
-        damping="0.1"
+        damping="0.0"
         friction="0.2" />
   </joint>

File: amr_description/urdf/amr_gazebo.xacro (robot description, xacro)
@@ -2,14 +2,14 @@
 <robot name="amr" xmlns:xacro="http://ros.org/wiki/xacro">
     <gazebo reference="back_wheel_right_side">
-  <material>
-    <friction>
-      <mu1>0.9</mu1>
-      <mu2>0.9</mu2>
-    </friction>
-    <surface>
-      <kp>100000.0</kp>
-      <kd>1.0</kd>
-    </surface>
-  </material>
+        <material>
+          <friction>
+            <mu1>1000000000.0</mu1>
+            <mu2>1000000000.0</mu2>
+          </friction>
+          <surface>
+            <kp>100000.0</kp>
+            <kd>1.0</kd>
+          </surface>
+        </material>
         <minDepth>0.001</minDepth>
         <maxVel>0.1</maxVel>
@@ -17,14 +17,14 @@
     </gazebo>
     <gazebo reference="back_wheel_left_side">
-  <material>
-    <friction>
-      <mu1>0.9</mu1>
-      <mu2>0.9</mu2>
-    </friction>
-    <surface>
-      <kp>100000.0</kp>
-      <kd>1.0</kd>
-    </surface>
-  </material>
+        <material>
+          <friction>
+            <mu1>1000000000.0</mu1>
+            <mu2>1000000000.0</mu2>
+          </friction>
+          <surface>
+            <kp>100000.0</kp>
+            <kd>1.0</kd>
+          </surface>
+        </material>
         <minDepth>0.001</minDepth>
         <maxVel>0.1</maxVel>
@@ -32,14 +32,14 @@
     </gazebo>
     <gazebo reference="middle_wheel_right_side">
-  <material>
-    <friction>
-      <mu1>0.9</mu1>
-      <mu2>0.9</mu2>
-    </friction>
-    <surface>
-      <kp>100000.0</kp>
-      <kd>1.0</kd>
-    </surface>
-  </material>
+        <material>
+          <friction>
+            <mu1>1000000000.0</mu1>
+            <mu2>1000000000.0</mu2>
+          </friction>
+          <surface>
+            <kp>100000.0</kp>
+            <kd>1.0</kd>
+          </surface>
+        </material>
         <minDepth>0.001</minDepth>
         <maxVel>0.1</maxVel>
@@ -47,14 +47,14 @@
     </gazebo>
     <gazebo reference="middle_wheel_left_side">
-  <material>
-    <friction>
-      <mu1>0.9</mu1>
-      <mu2>0.9</mu2>
-    </friction>
-    <surface>
-      <kp>100000.0</kp>
-      <kd>1.0</kd>
-    </surface>
-  </material>
+        <material>
+          <friction>
+            <mu1>1000000000.0</mu1>
+            <mu2>1000000000.0</mu2>
+          </friction>
+          <surface>
+            <kp>100000.0</kp>
+            <kd>1.0</kd>
+          </surface>
+        </material>
         <minDepth>0.001</minDepth>
         <maxVel>0.1</maxVel>
@@ -62,14 +62,14 @@
     </gazebo>
     <gazebo reference="front_wheel_right_side">
-  <material>
-    <friction>
-      <mu1>0.9</mu1>
-      <mu2>0.9</mu2>
-    </friction>
-    <surface>
-      <kp>100000.0</kp>
-      <kd>1.0</kd>
-    </surface>
-  </material>
+        <material>
+          <friction>
+            <mu1>1000000000.0</mu1>
+            <mu2>1000000000.0</mu2>
+          </friction>
+          <surface>
+            <kp>100000.0</kp>
+            <kd>1.0</kd>
+          </surface>
+        </material>
         <minDepth>0.001</minDepth>
         <maxVel>0.1</maxVel>
@@ -77,14 +77,14 @@
     </gazebo>
     <gazebo reference="front_wheel_left_side">
-  <material>
-    <friction>
-      <mu1>0.9</mu1>
-      <mu2>0.9</mu2>
-    </friction>
-    <surface>
-      <kp>100000.0</kp>
-      <kd>1.0</kd>
-    </surface>
-  </material>
+        <material>
+          <friction>
+            <mu1>1000000000.0</mu1>
+            <mu2>1000000000.0</mu2>
+          </friction>
+          <surface>
+            <kp>100000.0</kp>
+            <kd>1.0</kd>
+          </surface>
+        </material>
         <minDepth>0.001</minDepth>
         <maxVel>0.1</maxVel>
@@ -108,8 +108,8 @@
       <sensor name="imu" type="imu">
        <always_on>true</always_on>
-       <update_rate>50</update_rate>
+       <update_rate>100</update_rate>
        <gz_frame_id> imu_link</gz_frame_id>
        <topic>imu</topic>
-       <imu>
+       <!--imu>
         <angular_velocity>
           <x>
@@ -152,5 +152,5 @@
           </z>
         </linear_acceleration>
-       </imu>
+       </imu-->
       </sensor>
     </gazebo>

File: amr_description/urdf/amr_ros2_control.xacro (robot description, xacro)
@@ -53,4 +53,11 @@
             <state_interface name="velocity"/>
         </joint>
+        <joint name="del_box_connector">
+            <command_interface name= "position">
+                <param name="min">0</param>
+                <param name="max">0.890118</param>
+            </command_interface>
+            <state_interface name="position"/>
+        </joint>
     </ros2_control>
 </robot>

Commit message: Robot Enabled with turning

File: amr_description/urdf/amr.urdf.xacro (robot description, xacro)
@@ -34,5 +34,5 @@
         rpy="0 0 0" />
       <mass
-        value="1.001384" />
+        value="1.5" />
       <inertia
         ixx="8.726e-3"
@@ -54,5 +54,5 @@
       <origin
         xyz="0 0 0"
-        rpy="1.57 0 0" />
+        rpy="1.57 -0.071813801 0" />
       <geometry>
         <mesh
@@ -68,5 +68,5 @@
       <origin
         xyz="0 0 0"
-        rpy="1.57 0 0" />
+        rpy="1.57 -0.071813801 0" />
       <geometry>
         <mesh
@@ -108,5 +108,5 @@
       <origin
         xyz="0 0 0"
-        rpy="0 0 0" />
+        rpy="0 -0.071813801 0" />
       <geometry>
         <mesh
@@ -122,5 +122,5 @@
       <origin
         xyz="0 0 0"
-        rpy="0 0 0" />
+        rpy="0 -0.071813801 0" />
       <geometry>
         <mesh
@@ -248,4 +248,310 @@
   </joint>
   <link
+    name="front_right_connector">
+    <visual>
+      <origin
+        xyz="0 0 0"
+        rpy="0 0 0" />
+      <geometry>
+        <mesh
+          filename="package://amr_description/meshes/wconnector_right_side.stl" scale="0.001 0.001 0.001"/>
+      </geometry>
+      <material
+        name="">
+        <color
+          rgba="0.792156862745098 0.819607843137255 0.933333333333333 1" />
+      </material>
+    </visual>
+    <collision>
+      <origin
+        xyz="0 0 0"
+        rpy="0 0 0" />
+      <geometry>
+        <mesh
+          filename="package://amr_description/meshes/wconnector_right_side.stl" scale="0.001 0.001 0.001" />
+      </geometry>
+    </collision>
+    <inertial>
+      <origin
+        xyz="0 -0.005 0"
+        rpy="0 0 0" />
+      <mass
+        value="12.076e-3" />
+      <inertia
+        ixx="2.205e-6"
+        ixy="-4.149e-18"
+        ixz="-3.479e-14"
+        iyy="2.451457e-6"
+        iyz="-0.434e-9"
+        izz="3.35403e-7" />
+    </inertial>
+  </link>
+  <joint name="front_right_link_connector_joint" type="revolute">
+    <parent link="front_link_right_side"/>
+    <child link="front_right_connector"/>
+    <origin xyz="0.085041 -0.0065 -0.029463" rpy="0 0 0"/>
+    <axis xyz="0 0 1"/>
+      <limit
+        lower = "-3.14"
+        upper = "3.14"
+        effort="10000000"
+        velocity="10000000" />
+      <dynamics
+        damping="0.0"
+        friction="0.2" />
+  </joint>
+  <link
+    name="middle_right_connector">
+    <visual>
+      <origin
+        xyz="0 0 0"
+        rpy="0 0 0" />
+      <geometry>
+        <mesh
+          filename="package://amr_description/meshes/wconnector_right_side.stl" scale="0.001 0.001 0.001"/>
+      </geometry>
+      <material
+        name="">
+        <color
+          rgba="0.792156862745098 0.819607843137255 0.933333333333333 1" />
+      </material>
+    </visual>
+    <collision>
+      <origin
+        xyz="0 0 0"
+        rpy="0 0 0" />
+      <geometry>
+        <mesh
+          filename="package://amr_description/meshes/wconnector_right_side.stl" scale="0.001 0.001 0.001" />
+      </geometry>
+    </collision>
+    <inertial>
+      <origin
+        xyz="0 -0.005 0"
+        rpy="0 0 0" />
+      <mass
+        value="12.076e-3" />
+      <inertia
+        ixx="2.205e-6"
+        ixy="-4.149e-18"
+        ixz="-3.479e-14"
+        iyy="2.451457e-6"
+        iyz="-0.434e-9"
+        izz="3.35403e-7" />
+    </inertial>
+  </link>
+  <joint name="middle_right_link_connector_joint" type="fixed">
+    <parent link="front_link_right_side"/>
+    <child link="middle_right_connector"/>
+    <origin xyz="-0.069638 -0.0065 -0.039441" rpy="0 0 0"/>
+  </joint>
+  <link
+    name="back_right_connector">
+    <visual>
+      <origin
+        xyz="0 0 0"
+        rpy="0 0 0" />
+      <geometry>
+        <mesh
+          filename="package://amr_description/meshes/wconnector_right_side.stl" scale="0.001 0.001 0.001"/>
+      </geometry>
+      <material
+        name="">
+        <color
+          rgba="0.792156862745098 0.819607843137255 0.933333333333333 1" />
+      </material>
+    </visual>
+    <collision>
+      <origin
+        xyz="0 0 0"
+        rpy="0 0 0" />
+      <geometry>
+        <mesh
+          filename="package://amr_description/meshes/wconnector_right_side.stl" scale="0.001 0.001 0.001" />
+      </geometry>
+    </collision>
+    <inertial>
+      <origin
+        xyz="0 -0.005 0"
+        rpy="0 0 0" />
+      <mass
+        value="12.076e-3" />
+      <inertia
+        ixx="2.205e-6"
+        ixy="-4.149e-18"
+        ixz="-3.479e-14"
+        iyy="2.451457e-6"
+        iyz="-0.434e-9"
+        izz="3.35403e-7" />
+    </inertial>
+  </link>
+  <joint name="back_right_link_connector_joint" type="revolute">
+    <parent link="back_link_right_side"/>
+    <child link="back_right_connector"/>
+    <origin xyz="0 -0.0065 -0.039441" rpy="0 0 0"/>
+    <axis xyz="0 0 1"/>
+      <limit
+        lower = "-3.14"
+        upper = "3.14"
+        effort="10000000"
+        velocity="10000000" />
+      <dynamics
+        damping="0.0"
+        friction="0.2" />
+  </joint>
+  <link
+    name="front_left_connector">
+    <visual>
+      <origin
+        xyz="0 0 0"
+        rpy="0 0 0" />
+      <geometry>
+        <mesh
+          filename="package://amr_description/meshes/wconnector_left_side.stl" scale="0.001 0.001 0.001"/>
+      </geometry>
+      <material
+        name="">
+        <color
+          rgba="0.792156862745098 0.819607843137255 0.933333333333333 1" />
+      </material>
+    </visual>
+    <collision>
+      <origin
+        xyz="0 0 0"
+        rpy="0 0 0" />
+      <geometry>
+        <mesh
+          filename="package://amr_description/meshes/wconnector_left_side.stl" scale="0.001 0.001 0.001" />
+      </geometry>
+    </collision>
+    <inertial>
+      <origin
+        xyz="0 0.005 0"
+        rpy="0 0 0" />
+      <mass
+        value="12.076e-3" />
+      <inertia
+        ixx="2.205e-6"
+        ixy="-4.149e-18"
+        ixz="-3.479e-14"
+        iyy="2.451457e-6"
+        iyz="-0.434e-9"
+        izz="3.35403e-7" />
+    </inertial>
+  </link>
+  <joint name="front_left_link_connector_joint" type="revolute">
+    <parent link="front_link_left_side"/>
+    <child link="front_left_connector"/>
+    <origin xyz="0.085041 0.0065 -0.029463" rpy="0 0 0"/>
+    <axis xyz="0 0 1"/>
+      <limit
+        lower = "-3.14"
+        upper = "3.14"
+        effort="10000000"
+        velocity="10000000" />
+      <dynamics
+        damping="0.0"
+        friction="0.2" />
+  </joint>
+  <link
+    name="middle_left_connector">
+    <visual>
+      <origin
+        xyz="0 0 0"
+        rpy="0 0 0" />
+      <geometry>
+        <mesh
+          filename="package://amr_description/meshes/wconnector_left_side.stl" scale="0.001 0.001 0.001"/>
+      </geometry>
+      <material
+        name="">
+        <color
+          rgba="0.792156862745098 0.819607843137255 0.933333333333333 1" />
+      </material>
+    </visual>
+    <collision>
+      <origin
+        xyz="0 0 0"
+        rpy="0 0 0" />
+      <geometry>
+        <mesh
+          filename="package://amr_description/meshes/wconnector_left_side.stl" scale="0.001 0.001 0.001" />
+      </geometry>
+    </collision>
+    <inertial>
+      <origin
+        xyz="0 0.005 0"
+        rpy="0 0 0" />
+      <mass
+        value="12.076e-3" />
+      <inertia
+        ixx="2.205e-6"
+        ixy="-4.149e-18"
+        ixz="-3.479e-14"
+        iyy="2.451457e-6"
+        iyz="-0.434e-9"
+        izz="3.35403e-7" />
+    </inertial>
+  </link>
+  <joint name="middle_left_link_connector_joint" type="fixed">
+    <parent link="front_link_left_side"/>
+    <child link="middle_left_connector"/>
+    <origin xyz="-0.069638 0.0065 -0.039441" rpy="0 0 0"/>
+  </joint>
+  <link
+    name="back_left_connector">
+    <visual>
+      <origin
+        xyz="0 0 0"
+        rpy="0 0 0" />
+      <geometry>
+        <mesh
+          filename="package://amr_description/meshes/wconnector_left_side.stl" scale="0.001 0.001 0.001"/>
+      </geometry>
+      <material
+        name="">
+        <color
+          rgba="0.792156862745098 0.819607843137255 0.933333333333333 1" />
+      </material>
+    </visual>
+    <collision>
+      <origin
+        xyz="0 0 0"
+        rpy="0 0 0" />
+      <geometry>
+        <mesh
+          filename="package://amr_description/meshes/wconnector_left_side.stl" scale="0.001 0.001 0.001" />
+      </geometry>
+    </collision>
+    <inertial>
+      <origin
+        xyz="0 0.005 0"
+        rpy="0 0 0" />
+      <mass
+        value="12.076e-3" />
+      <inertia
+        ixx="2.205e-6"
+        ixy="-4.149e-18"
+        ixz="-3.479e-14"
+        iyy="2.451457e-6"
+        iyz="-0.434e-9"
+        izz="3.35403e-7" />
+    </inertial>
+  </link>
+  <joint name="back_left_link_connector_joint" type="revolute">
+    <parent link="back_link_left_side"/>
+    <child link="back_left_connector"/>
+    <origin xyz="0 0.0065 -0.039441" rpy="0 0 0"/>
+    <axis xyz="0 0 1"/>
+      <limit
+        lower = "-3.14"
+        upper = "3.14"
+        effort="10000000"
+        velocity="10000000" />
+      <dynamics
+        damping="0.0"
+        friction="0.2" />
+  </joint>
+  <link
     name="back_wheel_right_side">
     <visual>
@@ -288,7 +594,7 @@
   </link>
   <joint name="back_right_wheel_revolute" type="continuous">
-    <parent link="back_link_right_side"/>
+    <parent link="back_right_connector"/>
     <child link="back_wheel_right_side"/>
-    <origin xyz="0 -0.0065 -0.03514" rpy="0 0 0"/>
+    <origin xyz="0 -0.010 0" rpy="0 0 0"/>
     <axis xyz="0 1 0"/>
     <limit
@@ -340,7 +646,7 @@
   </link>
   <joint name="back_left_wheel_revolute" type="continuous">
-    <parent link="back_link_left_side"/>
+    <parent link="back_left_connector"/>
     <child link="back_wheel_left_side"/>
-    <origin xyz="0 0.0065 -0.03514" rpy="0 0 0"/>
+    <origin xyz="0 0.010 0" rpy="0 0 0"/>
     <axis xyz="0 1 0"/>
     <limit
@@ -392,7 +698,7 @@
   </link>
   <joint name="middle_left_wheel_revolute" type="continuous">
-    <parent link="front_link_left_side"/>
+    <parent link="middle_left_connector"/>
     <child link="middle_wheel_left_side"/>
-    <origin xyz="-0.072288 0.0065 -0.034343" rpy="0 0 0"/>
+    <origin xyz="0 0.010 0" rpy="0 0 0"/>
     <axis xyz="0 1 0"/>
     <limit
@@ -444,7 +750,7 @@
   </link>
   <joint name="middle_right_wheel_revolute" type="continuous">
-    <parent link="front_link_right_side"/>
+    <parent link="middle_right_connector"/>
     <child link="middle_wheel_right_side"/>
-    <origin xyz="-0.072288 -0.0065 -0.034343" rpy="0 0 0"/>
+    <origin xyz="0 -0.01 0" rpy="0 0 0"/>
     <axis xyz="0 1 0"/>
     <limit
@@ -496,7 +802,7 @@
   </link>
   <joint name="front_left_wheel_revolute" type="continuous">
-    <parent link="front_link_left_side"/>
+    <parent link="front_left_connector"/>
     <child link="front_wheel_left_side"/>
-    <origin xyz="0.082708 0.0065 -0.035489" rpy="0 0 0"/>
+    <origin xyz="0 0.010 0" rpy="0 0 0"/>
     <axis xyz="0 1 0"/>
     <limit
@@ -548,7 +854,7 @@
   </link>
   <joint name="front_right_wheel_revolute" type="continuous">
-    <parent link="front_link_right_side"/>
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
File: amr_description/urdf/amr_ros2_control.xacro (robot description, xacro)
@@ -53,4 +53,32 @@
             <state_interface name="velocity"/>
         </joint>
+        <joint name="front_left_link_connector_joint">
+            <command_interface name= "position">
+                <param name="min">-3.14</param>
+                <param name="max">3.14</param>
+            </command_interface>
+            <state_interface name="position"/>
+        </joint>
+        <joint name="front_right_link_connector_joint">
+            <command_interface name= "position">
+                <param name="min">-3.14</param>
+                <param name="max">3.14</param>
+            </command_interface>
+            <state_interface name="position"/>
+        </joint>
+        <joint name="back_left_link_connector_joint">
+            <command_interface name= "position">
+                <param name="min">-3.14</param>
+                <param name="max">3.14</param>
+            </command_interface>
+            <state_interface name="position"/>
+        </joint>
+        <joint name="back_right_link_connector_joint">
+            <command_interface name= "position">
+                <param name="min">-3.14</param>
+                <param name="max">3.14</param>
+            </command_interface>
+            <state_interface name="position"/>
+        </joint>
         <joint name="del_box_connector">
             <command_interface name= "position">

Commit message: Updated files and made changes

File: amr_description/urdf/amr.urdf.xacro (robot description, xacro)
@@ -47,5 +47,5 @@
     <parent link="base_footprint"/>
     <child link="base_link"/>
-    <origin xyz="0 0 0.09" rpy="0 0 0"/>
+    <origin xyz="0.00037 0 0.0803" rpy="0 0 0"/>
   </joint>
   <link
@@ -866,5 +866,13 @@
   </joint>
   <link name="imu_link">
-    <visual>
+    <inertial>
+      <origin xyz="-0.00552433659106688 0.000168210391520346 0.000514000497342681" rpy="0 0 0" />
+      <mass value="0.000528415362211671" />
+      <inertia ixx="1.46176048428261E-08" ixy="1.40015117949421E-10" ixz="-1.99633872937403E-12"
+               iyy="8.59662482954888E-09" iyz="7.52375112767959E-12"
+               izz="2.30279421279312E-08" />
+    </inertial>
+    <visual>
+      <origin xyz="0 0 0" rpy="0 0 0" />
       <geometry>
         <box size="0.02 0.02 0.005"/>
@@ -878,5 +886,5 @@
       <parent link="base_link"/>
       <child link="imu_link"/>
-      <origin xyz="0 0 0.005" rpy="0 0 0"/>
+      <origin xyz="0.00037 0 0.005" rpy="0 0 0"/>
       <axis xyz="0 0 0"/>
   </joint>

File: amr_description/urdf/amr_gazebo.xacro (robot description, xacro)
@@ -111,5 +111,5 @@
        <gz_frame_id> imu_link</gz_frame_id>
        <topic>imu</topic>
-       <imu>
+       <!--imu>
         <angular_velocity>
           <x>
@@ -152,5 +152,5 @@
           </z>
         </linear_acceleration>
-       </imu>
+       </imu-->
       </sensor>
     </gazebo>
