Commit message: Odometry Configured Perfectly

File: amr_description/urdf/amr.urdf.xacro (robot description, xacro)
@@ -14,8 +14,6 @@
           filename="package://amr_description/meshes/base_link.stl" scale="0.001 0.001 0.001"/>
       </geometry>
-      <material
-        name="">
-        <color
-          rgba="0.792156862745098 0.819607843137255 0.933333333333333 1" />
+      <material name="aluminum_silver">
+        <color rgba="0.8 0.85 0.88 1.0"/>
       </material>
     </visual>
@@ -59,8 +57,6 @@
           filename="package://amr_description/meshes/front_link_right_side.stl" scale="0.001 0.001 0.001"/>
       </geometry>
-      <material
-        name="">
-        <color
-          rgba="0.792156862745098 0.819607843137255 0.933333333333333 1" />
+      <material name="connector_black">
+        <color rgba="0.1 0.1 0.1 1.0"/>
       </material>
     </visual>
@@ -113,8 +109,6 @@
           filename="package://amr_description/meshes/front_link_left_side.stl" scale="0.001 0.001 0.001"/>
       </geometry>
-      <material
-        name="">
-        <color
-          rgba="0.792156862745098 0.819607843137255 0.933333333333333 1" />
+      <material name="connector_black">
+        <color rgba="0.1 0.1 0.1 1.0"/> <!-- Matte black -->
       </material>
     </visual>
@@ -167,8 +161,6 @@
           filename="package://amr_description/meshes/back_link_left_side.stl" scale="0.001 0.001 0.001"/>
       </geometry>
-      <material
-        name="">
-        <color
-          rgba="0.792156862745098 0.819607843137255 0.933333333333333 1" />
+      <material name="connector_black">
+        <color rgba="0.1 0.1 0.1 1.0"/>
       </material>
     </visual>
@@ -212,8 +204,6 @@
           filename="package://amr_description/meshes/back_link_right_side.stl" scale="0.001 0.001 0.001"/>
       </geometry>
-      <material
-        name="">
-        <color
-          rgba="0.792156862745098 0.819607843137255 0.933333333333333 1" />
+      <material name="connector_black">
+        <color rgba="0.1 0.1 0.1 1.0"/>
       </material>
     </visual>
@@ -563,8 +553,6 @@
           filename="package://amr_description/meshes/back_wheel_right_side.stl" scale="0.001 0.001 0.001"/>
       </geometry>
-      <material
-        name="">
-        <color
-          rgba="0.792156862745098 0.819607843137255 0.933333333333333 1" />
+      <material name="rubber_black">
+        <color rgba="0.2 0.2 0.2 1.0"/>
       </material>
     </visual>
@@ -615,8 +603,6 @@
           filename="package://amr_description/meshes/back_wheel_left_side.stl" scale="0.001 0.001 0.001"/>
       </geometry>
-      <material
-        name="">
-        <color
-          rgba="0.792156862745098 0.819607843137255 0.933333333333333 1" />
+      <material name="rubber_black">
+        <color rgba="0.2 0.2 0.2 1.0"/>
       </material>
     </visual>
@@ -667,8 +653,6 @@
           filename="package://amr_description/meshes/middle_wheel_left_side.stl" scale="0.001 0.001 0.001"/>
       </geometry>
-      <material
-        name="">
-        <color
-          rgba="0.792156862745098 0.819607843137255 0.933333333333333 1" />
+      <material name="rubber_black">
+        <color rgba="0.2 0.2 0.2 1.0"/>
       </material>
     </visual>
@@ -719,8 +703,6 @@
           filename="package://amr_description/meshes/middle_wheel_right_side.stl" scale="0.001 0.001 0.001"/>
       </geometry>
-      <material
-        name="">
-        <color
-          rgba="0.792156862745098 0.819607843137255 0.933333333333333 1" />
+      <material name="rubber_black">
+        <color rgba="0.2 0.2 0.2 1.0"/>
       </material>
     </visual>
@@ -771,8 +753,6 @@
           filename="package://amr_description/meshes/front_wheel_left_side.stl" scale="0.001 0.001 0.001"/>
       </geometry>
-      <material
-        name="">
-        <color
-          rgba="0.792156862745098 0.819607843137255 0.933333333333333 1" />
+      <material name="rubber_black">
+        <color rgba="0.2 0.2 0.2 1.0"/>
       </material>
     </visual>
@@ -823,8 +803,6 @@
           filename="package://amr_description/meshes/front_wheel_right_side.stl" scale="0.001 0.001 0.001"/>
       </geometry>
-      <material
-        name="">
-        <color
-          rgba="0.792156862745098 0.819607843137255 0.933333333333333 1" />
+      <material name="rubber_black">
+        <color rgba="0.2 0.2 0.2 1.0"/>
       </material>
     </visual>
@@ -1035,8 +1013,6 @@
           filename="package://amr_description/meshes/delivery_box_wol.stl" scale="0.001 0.001 0.001"/>
       </geometry>
-      <material
-        name="">
-        <color
-          rgba="0.792156862745098 0.819607843137255 0.933333333333333 1" />
+      <material name="delivery_box_blue">
+        <color rgba="0.2 0.4 0.8 1.0"/>  <!-- A strong cobalt blue -->
       </material>
     </visual>

File: amr_description/urdf/amr_gazebo.xacro (robot description, xacro)
@@ -2,92 +2,116 @@
 <robot name="amr" xmlns:xacro="http://ros.org/wiki/xacro">
     <gazebo reference="back_wheel_right_side">
-        <material>
-          <friction>
-            <mu1>1000000000.0</mu1>
-            <mu2>1000000000.0</mu2>
-          </friction>
-          <surface>
-            <kp>100000.0</kp>
-            <kd>1.0</kd>
-          </surface>
-        </material>
-        <minDepth>0.001</minDepth>
-        <maxVel>0.1</maxVel>
-        <fdir1>1 0 0</fdir1>
+      <surface>
+        <friction>
+          <ode>
+            <mu>1000000.0</mu>
+            <mu2>1000000.0</mu2>
+          </ode>
+        </friction>
+        <contact>
+          <ode>
+            <kp>500000.0</kp>
+            <kd>5.0</kd>
+            <min_depth>0.001</min_depth>
+            <max_vel>0.1</max_vel>
+          </ode>
+        </contact>
+      </surface>
+      <fdir1>1 0 0</fdir1>
     </gazebo>
     <gazebo reference="back_wheel_left_side">
-        <material>
-          <friction>
-            <mu1>1000000000.0</mu1>
-            <mu2>1000000000.0</mu2>
-          </friction>
-          <surface>
-            <kp>100000.0</kp>
-            <kd>1.0</kd>
-          </surface>
-        </material>
-        <minDepth>0.001</minDepth>
-        <maxVel>0.1</maxVel>
-        <fdir1>1 0 0</fdir1>
+      <surface>
+        <friction>
+          <ode>
+            <mu>1000000.0</mu>
+            <mu2>1000000.0</mu2>
+          </ode>
+        </friction>
+        <contact>
+          <ode>
+            <kp>500000.0</kp>
+            <kd>5.0</kd>
+            <min_depth>0.001</min_depth>
+            <max_vel>0.1</max_vel>
+          </ode>
+        </contact>
+      </surface>
+      <fdir1>1 0 0</fdir1>
     </gazebo>
     <gazebo reference="middle_wheel_right_side">
-        <material>
-          <friction>
-            <mu1>1000000000.0</mu1>
-            <mu2>1000000000.0</mu2>
-          </friction>
-          <surface>
-            <kp>100000.0</kp>
-            <kd>1.0</kd>
-          </surface>
-        </material>
-        <minDepth>0.001</minDepth>
-        <maxVel>0.1</maxVel>
-        <fdir1>1 0 0</fdir1>
+      <surface>
+        <friction>
+          <ode>
+            <mu>1000000.0</mu>
+            <mu2>1000000.0</mu2>
+          </ode>
+        </friction>
+        <contact>
+          <ode>
+            <kp>500000.0</kp>
+            <kd>5.0</kd>
+            <min_depth>0.001</min_depth>
+            <max_vel>0.1</max_vel>
+          </ode>
+        </contact>
+      </surface>
+      <fdir1>1 0 0</fdir1>
     </gazebo>
     <gazebo reference="middle_wheel_left_side">
-        <material>
-          <friction>
-            <mu1>1000000000.0</mu1>
-            <mu2>1000000000.0</mu2>
-          </friction>
-          <surface>
-            <kp>100000.0</kp>
-            <kd>1.0</kd>
-          </surface>
-        </material>
-        <minDepth>0.001</minDepth>
-        <maxVel>0.1</maxVel>
-        <fdir1>1 0 0</fdir1>
+      <surface>
+        <friction>
+          <ode>
+            <mu>1000000.0</mu>
+            <mu2>1000000.0</mu2>
+          </ode>
+        </friction>
+        <contact>
+          <ode>
+            <kp>500000.0</kp>
+            <kd>5.0</kd>
+            <min_depth>0.001</min_depth>
+            <max_vel>0.1</max_vel>
+          </ode>
+        </contact>
+      </surface>
+      <fdir1>1 0 0</fdir1>
     </gazebo>
     <gazebo reference="front_wheel_right_side">
-        <material>
-          <friction>
-            <mu1>1000000000.0</mu1>
-            <mu2>1000000000.0</mu2>
-          </friction>
-          <surface>
-            <kp>100000.0</kp>
-            <kd>1.0</kd>
-          </surface>
-        </material>
-        <minDepth>0.001</minDepth>
-        <maxVel>0.1</maxVel>
-        <fdir1>1 0 0</fdir1>
+      <surface>
+        <friction>
+          <ode>
+            <mu>1000000.0</mu>
+            <mu2>1000000.0</mu2>
+          </ode>
+        </friction>
+        <contact>
+          <ode>
+            <kp>500000.0</kp>
+            <kd>5.0</kd>
+            <min_depth>0.001</min_depth>
+            <max_vel>0.1</max_vel>
+          </ode>
+        </contact>
+      </surface>
+      <fdir1>1 0 0</fdir1>
     </gazebo>
     <gazebo reference="front_wheel_left_side">
-        <material>
-          <friction>
-            <mu1>1000000000.0</mu1>
-            <mu2>1000000000.0</mu2>
-          </friction>
-          <surface>
-            <kp>100000.0</kp>
-            <kd>1.0</kd>
-          </surface>
-        </material>
-        <minDepth>0.001</minDepth>
-        <maxVel>0.1</maxVel>
-        <fdir1>1 0 0</fdir1>
+      <surface>
+        <friction>
+          <ode>
+            <mu>1000000.0</mu>
+            <mu2>1000000.0</mu2>
+          </ode>
+        </friction>
+        <contact>
+          <ode>
+            <kp>500000.0</kp>
+            <kd>5.0</kd>
+            <min_depth>0.001</min_depth>
+            <max_vel>0.1</max_vel>
+          </ode>
+        </contact>
+      </surface>
+      <fdir1>1 0 0</fdir1>
     </gazebo>
     <gazebo>
